File: picoruby-tea5767-plan/fm_spectrum_monitor.kicad_sch (KiCad schematic)
At the start: 2 parts, among them U1 RPi_Pico, U2 TEA5767

Commit message: docs: PR #2 review feedback への対応一括（CodeRabbit + reviewdog）
CodeRabbit 4 件:
- CR-1 (Major): docs/notes/2026-04-23-display-architecture.md の file:// 矛盾を解消．
  ローカル開発は http://localhost 前提に統一し，README L417-418 の CORS 制約と整合．
- CR-2 (Major): fm_spectrum_monitor.kicad_sch の全 passive ピンを電気的役割に応じた
  type へ修正．I2C 双方向ピンを bidirectional，電源入力を power_in，3V3OUT を
  power_out，L_OUT/R_OUT を output に変更（ANT は受動端子のため passive 維持）．
  これにより KiCad ERC が誤接続を検出できるようになる．
- CR-3 (Trivial): USB_CDC_TO_BROWSER ラベルが配線上にないためグラフィック text に変更．
- CR-4 (Trivial): 「開くことができる」を「開ける」に簡潔化（C5 と統合）．

reviewdog 機械的修正 6 件 (採用):
- L36 arabic-kanji-numbers: もう一つ → もう 1 つ
- L136 prh js→JavaScript: Ruby.wasm + js → Ruby.wasm + JavaScript
- L195 ja-no-redundant-expression: 指定を行う → 指定する
- L227 prh ユーザ→ユーザー: ユーザ体験 → ユーザー体験
- L428, L437 ja-no-space-around-parentheses: ** ＋ （ の競合を rewrite で解消

reviewdog 文章書き換え 6 件 (採用):
- C1 (L5 sentence-length 132): 1 文を 2 文に分割
- C2 (L39 sentence-length 104): 3 文に分割
- C3 (L174 sentence-length 108): 主述を分けて短文化
- C4 (L34 no-doubled-joshi が連続): 助詞を変えて句読点で区切り
- C5 (L123 no-doubled-joshi で連続): 主述を分離（CR-4 と統合）
- C6 (L176 no-doubled-joshi も連続): 「Pico も…ブラウザも」を「Pico や実ブラウザがなくても」に

reviewdog 18 件は別途返信で却下方針:
- prh JS 8 件: JSON のサブストリング誤検出．中央 prh.yml の word boundary 不備
  （tomio2480/github-workflows#12 で対応）
- ja-no-mixed-period 8 件: 表/図キャプションは sentence でないため `．` を付けない
- sentence-length 2 件: 長尺 alt text は a11y のため許容

Co-Authored-By: Claude Opus 4.7 (1M context) <noreply@anthropic.com>
Other:
- note added: "USB_CDC_TO_BROWSER"
Changed lines of the file:
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@@
   (effects (font (size 1.27 1.27)) (justify left bottom))
 )
-(label "USB_CDC_TO_BROWSER" (at 95 70 0)
+(text "USB_CDC_TO_BROWSER" (at 95 70 0)
   (effects (font (size 1.27 1.27)) (justify left bottom))
 )
